File: Electronics/OpenThereminV45.kicad_sch (KiCad schematic)
At the start: 99 parts, among them J1 USB_C_Receptacle 12401610E4#2A, J2 Conn_02x03_Odd_Even, J3 Conn_02x05_Odd_Even, P1 10k, P10 BUTTON, P11 A3_PAD, P12 A2_PAD, P13 A1_PAD, P14 A0_PAD, P16 GND, P2 10k, P3 10k, P4 10k, P8 VCC, P9 GND, U1 TTP223, U10 CH340C, U11 LP2985-3.3, U12 MCP4922-E/SL, U2 74HC4060D, U3 74HC4060D, U4 74HC74, U5 HEF4069, U6 MCP4921-E/SN, U7 MCP4922-E/SL, U8 MCP6002T-I/SN, U9 ATmega328P-AU, X1 16MHz, X2 7.3721MHz, Y1 MountPad3, Y2 MountPad3, Y3 PLUG_3_5_SMD SJ-3502-SMT-TR, Y7 PLUG_3_5_SMD SJ-3502-SMT-TR

Commit message: Update schema
- Re-organize schema layout
- Move DNP info from text description to part attribute
- Move PN info from text description to part attribute
- Fix I/O attribute for some pins and labels
- Add NC labels for unused pins
- Added LCSC, Vendor and PN info for most parts
Parts:
- removed L1: 1mH CC453232A-102KL, GaudiLabsFootPrints:COIL_T, symbol OpenThereminV41-rescue:FILTER-OpenThereminV4-rescue
- removed Y7: PLUG_3_5_SMD SJ-3502-SMT-TR, GaudiLabsFootPrints:SJ-3502-SMT-TR, symbol OpenThereminV41-rescue:PLUG_3_5_SMD-OpenThereminV4-rescue
- added L3: 1mH, GaudiLabsFootPrints:COIL_T, symbol OpenThereminV41-rescue:FILTER-OpenThereminV4-rescue
- added Y4: PLUG_3_5_SMD, GaudiLabsFootPrints:SJ-3502-SMT-TR, symbol OpenThereminV41-rescue:PLUG_3_5_SMD-OpenThereminV4-rescue
- C1, C10, C2, C3, C7, C8, C9: value 150pF -> 150p; LCSC (none) -> C107038; Note (none) -> C0G/N0P; PN (none) -> CC0603JRNPO9BN151; Vendor (none) -> YAGEO
- C11: LCSC (none) -> C376764; Note (none) -> C0G/N0P; PN (none) -> TCC0603COG100J500CT; Vendor (none) -> CCTC
- C12, C5: value 470pF -> 470p; LCSC (none) -> C106211; Note (none) -> C0G/N0P; PN (none) -> CC0603JRNPO9BN471; Vendor (none) -> YAGEO
- C13, C23, C24, C25, C26, C27, C28, C6: value 100nF -> 100n; LCSC (none) -> C282519; PN (none) -> TCC0603X7R104K500CT; Vendor (none) -> CCTC
- C14: value 47pF -> 47p; LCSC (none) -> C94904; Note (none) -> C0G/N0P; PN (none) -> 0603CG470J500NT; Vendor (none) -> FH
- C15, C16, C34: value 22pF -> 22p; LCSC (none) -> C105620; Note (none) -> C0G/N0P; PN (none) -> CC0603JRNPO9BN220; Vendor (none) -> YAGEO
- C17, C18: value 22pF -> 30p; LCSC (none) -> C107047; Note (none) -> C0G/N0P; PN (none) -> CC0603JRNPO9BN330; Vendor (none) -> YAGEO
- C20, C21, C30, C32, C33, C35: LCSC (none) -> C282519; PN (none) -> TCC0603X7R104K500CT; Vendor (none) -> CCTC
- C22, C38: LCSC (none) -> C376807; PN (none) -> TCC0603X7R103M500CT; Vendor (none) -> CCTC
- C29: value 10uF -> 10u; LCSC (none) -> C1691; PN (none) -> CL10A106MQ8NNNC; Vendor (none) -> Samsung
- C36, C37: LCSC (none) -> C1691; PN (none) -> CL10A106MQ8NNNC; Vendor (none) -> Samsung
- C4: value not assembled -> ~; now not fitted; now left out of the parts list
- D3: value DualLED 156125RB73000 -> DualLED; PN (none) -> 156125RB73000
- GROUND1, P10, P11, P12, P13, P14, P16, P8, P9, W1, W2: now left out of the parts list
- J1: value USB_C_Receptacle 12401610E4#2A -> USB_C_Receptacle 12401610E4#2A
- J2, J3: now not fitted
- L2: value 1mH CC453232A-102KL -> 1mH; LCSC (none) -> C394145; PN (none) -> FHW1812IF102KST; Vendor (none) -> FH
- P1, P2, P3, P4: PN (none) -> PS15NV60-103A3030
- R1, R11, R13, R5: LCSC (none) -> C322165; Note (none) -> 1%; PN (none) -> RS-03L4704FT; Vendor (none) -> FH
- R10, R2, R20, R6, R9: LCSC (none) -> C294652; Note (none) -> 1%; PN (none) -> RS-03K2201FT; Vendor (none) -> FH
- R12, R14, R18, R19: LCSC (none) -> C116694; Note (none) -> 1%; PN (none) -> RS-03K4700FT; Vendor (none) -> FH
- R15, R16, R3, R4, R7, R8: LCSC (none) -> C3152121; Note (none) -> 1%; PN (none) -> SC0603F1003F2BNRH; Vendor (none) -> Sunway
- R21, R22: LCSC (none) -> C3152148; Note (none) -> 1%; PN (none) -> SC0603F5101F2BNRH; Vendor (none) -> Sunway
- U1: LCSC (none) -> C5345654; PN (none) -> HK2301; Vendor (none) -> Hichon
- U10: LCSC (none) -> C84681; PN (none) -> CH340C; Vendor (none) -> WCH
- U11: LCSC (none) -> C95414; PN (none) -> LP2985-33DBVR; Vendor (none) -> Ti
- U12, U7: LCSC (none) -> C39851; PN (none) -> MCP4922-E/SL; Vendor (none) -> Microchip
- U2, U3: LCSC (none) -> C5649; PN (none) -> 74HC4060D,653; Vendor (none) -> Nexperia
- U4: LCSC (none) -> C27597; PN (none) -> 74HC74D,653; Vendor (none) -> Nexperia
- U5: LCSC (none) -> C6739; PN (none) -> HEF4069UBT,653; Vendor (none) -> Nexperia
- U6: LCSC (none) -> C43499; PN (none) -> MCP4921-E/SN; Vendor (none) -> Microchip
- U8: LCSC (none) -> C20538868; PN (none) -> MCP6002T-I/SN(MS); Vendor (none) -> MSKSEMI
- U9: LCSC (none) -> C14877; PN (none) -> ATmega328P-AU; Vendor (none) -> Microchip
- X1: LCSC (none) -> C7473031; Note (none) -> 15~18pF; PN (none) -> M49SMD16M15PF15PPM; Vendor (none) -> SST
- X2: value 7.3721MHz -> 7.3728MHz; LCSC (none) -> C19173022; Note (none) -> 20pF; PN (none) -> RC07372602; Vendor (none) -> TROQ
- Y1: value MountPad3 -> Pitch
- Y2: value MountPad3 -> Volume
- Y3: value PLUG_3_5_SMD SJ-3502-SMT-TR -> PLUG_3_5_SMD; PN (none) -> SJ-3502-SMT-TR
Connections:
- net AUDIO: now also Y4.3 (L)
- net GATE: now also Y4.2 (R)
- net GND: now also Y4.1 (GND)
- net at C2.1, C4.1, C5.1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: now also L3.1
- net at C1.1, C14.1, R2.1: now also L3.2
- no-connect marks 0 -> 44
Other:
- note added: "CV & audio output"
- note added: "Control input"
- note added: "Debug"
- note added: "MCU"
- note added: "PWR"
- note added: "Pitch & volume input"
- note added: "USB-C & USB to serial"
- note removed: "PS15NV60-103A3030"
- moved on the sheet: C1, C10, C11, C12, C13, C14, C15, C16, C17, C18, C2, C20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

Commit message: Update schema & layout
- Adjust layout base on JLC capabilities
- Re-do USB layout
- Replace 3.5mm jack, inductor, type-c connector and LED with higher availability option
- Add 5x5mm SN block
- Remove some logos and text for personal preference
Parts:
- removed D3: DualLED, GaudiLabsFootPrints:WL-SBRW, symbol GaudiLabsPartsLibrary:DualLED
- removed J1: USB_C_Receptacle 12401610E4#2A, GaudiLabsFootPrints:USB_C_Receptacle_Amphenol_12401610E4-2A, symbol GaudiLabsPartsLibrary:USB_C_Receptacle
- removed Y3, Y4: PLUG_3_5_SMD, GaudiLabsFootPrints:SJ-3502-SMT-TR, symbol OpenThereminV41-rescue:PLUG_3_5_SMD-OpenThereminV4-rescue
- added D3: LTST-C235KGKRKT, LED_SMD:LED_LiteOn_LTST-C235KGKRKT, symbol LED:LTST-C235KGKRKT
- added J4, J5: PJ-320B, Library:XKB_PJ-320B, symbol Connector_Audio:AudioJack3
- added J6: USB_C_Receptacle_USB2.0_16P, Connector_USB:USB_C_Receptacle_GCT_USB4105-xx-A_16P_TopMnt_Horizontal, symbol Connector:USB_C_Receptacle_USB2.0_16P
- D1, D2: LCSC (none) -> C3272485; PN (none) -> BB914E6327HTSA1; Vendor (none) -> Infineon
- L1: renamed from L3; footprint GaudiLabsFootPrints:COIL_T -> Inductor_SMD:L_1812_4532Metric
- L2: footprint GaudiLabsFootPrints:COIL_T -> Inductor_SMD:L_1812_4532Metric
- P1, P2, P3, P4: LCSC (none) -> C5848081; Vendor (none) -> Amphenol
- R17: LCSC (none) -> C3152123; PN (none) -> SC0603F1002F2BNRH; Vendor (none) -> Sunway
- Y1, Y2: now left out of the parts list
Connections:
- net AUDIO: now also J5.T
- net CV1: now also J4.R
- net CV2: now also J4.T
- net D+: now also J6.A6 (D+), J6.B6 (D+); no longer J3.9 (Pin_9)
- net D-: now also J6.A7 (D-), J6.B7 (D-); no longer J3.8 (Pin_8)
- net GATE: now also J5.R
- net GND: now also D3.1 (K2), D3.4 (K1), J4.S, J5.S, J6.A1 (GND), J6.A12 (GND), J6.B1 (GND), J6.B12 (GND), J6.S1 (SHIELD)
- net VCC: now also J6.A4 (VBUS), J6.A9 (VBUS), J6.B4 (VBUS), J6.B9 (VBUS)
- net VoutA: now reaches R4.2, U7.14 (VoutA)
- net at R18.1: now also D3.2 (A2)
- net at R19.1: now also D3.3 (A1)
- net at R21.1: now also J6.A5 (CC1)
- net at R22.1: now also J6.B5 (CC2)
- net LED_BLUE renamed LED_GREEN
- no-connect marks 44 -> 37
Other:
- moved on the sheet: C1, C10, C11, C12, C13, C14, C15, C16, C17, C18, C2, C20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
